Commit message: split urdfs to have gazebo or isaac ros2 control

File: src/lerobot_description/urdf/so101_ros2_control_gazebo.xacro (robot description, xacro)
@@ -1,4 +1,10 @@
 <?xml version="1.0"?>
 <robot xmlns:xacro="http://www.ros.org/wiki/xacro">
+    <!-- ROS 2 Control -->
+    <gazebo>
+        <plugin filename="gz_ros2_control-system" name="gz_ros2_control::GazeboSimROS2ControlPlugin">
+            <parameters>$(find lerobot_controller)/config/so101_controllers.yaml</parameters>
+        </plugin>
+    </gazebo>
     <ros2_control name="RobotSystem" type="system">
         <!-- ros2_control Gazebo -->
@@ -6,5 +12,5 @@
             <plugin>gz_ros2_control/GazeboSimSystem</plugin>
         </hardware>
-        <joint name="1">
+        <joint name="shoulder_pan">
             <command_interface name="position">
                 <param name="min">-1.91986</param>
@@ -13,5 +19,5 @@
             <state_interface name="position" />
         </joint>
-        <joint name="2">
+        <joint name="shoulder_lift">
             <command_interface name="position">
                 <param name="min">-1.74533</param>
@@ -20,5 +26,5 @@
             <state_interface name="position" />
         </joint>
-        <joint name="3">
+        <joint name="elbow_flex">
             <command_interface name="position">
                 <param name="min">-1.74533</param>
@@ -27,5 +33,5 @@
             <state_interface name="position" />
         </joint>
-        <joint name="4">
+        <joint name="wrist_flex">
             <command_interface name="position">
                 <param name="min">-1.65806</param>
@@ -34,5 +40,5 @@
             <state_interface name="position" />
         </joint>
-        <joint name="5">
+        <joint name="wrist_roll">
             <command_interface name="position">
                 <param name="min">-2.79253</param>
@@ -41,5 +47,5 @@
             <state_interface name="position" />
         </joint>
-        <joint name="6">
+        <joint name="gripper">
             <command_interface name="position">
                 <param name="min">-0.174533</param>
